File: Hardware/LilyPad SimplePower_45_degree_for_panelization.brd (EAGLE design)
At the start: 28.4 x 28.4 mm, 22 parts, among them U1 MCP73831

Commit message: Updating polygon to GND layer
Routing:
- added copper zone on layer 1, net GND
- added copper zone on layer 16, net GND
- removed copper zone on layer 1, net N$2
- removed copper zone on layer 16, net N$8
